File: Rotavap/Pressure-control/Pressure-control/Pressure-control.sch (KiCad schematic (older format))
At the start: 8 parts, among them P1 Power, P2 Analog, P3 Digital, P4 Digital, P5 CONN_01X01, P6 CONN_01X01, P7 CONN_01X01, P8 CONN_01X01

Commit message: Update Pressure-control.sch
Parts:
- added D1: 1N4007, Diode_THT:D_DO-41_SOD81_P10.16mm_Horizontal, symbol Diode:1N4007
- added D?: LED, symbol Device:LED
- added K1: 833H-1C-C 12V DC, Relay_THT:Relay_StandexMeder_DIP_LowProfile, symbol Relay:DIPxx-1Cxx-51x
- added M?: Motor_AC, symbol Motor:Motor_AC
- added Q1: BC547, Package_TO_SOT_THT:TO-92_Inline, symbol Transistor_BJT:BC547
- added R1, R2: 1000, symbol Device:R
- added U1: EL814, symbol Isolator:EL814
Connections:
- net 13(SCK): now also R1.2
- net GND: now also D?.1 (K), Q1.3 (E)
- new net: R1.1, U1.1
- new net: D?.2 (A), U1.2
- new net: R2.1, U1.3
- new net: D1.2 (A), K1.6, Q1.1 (C)
- new net: K1.7, K1.8, M?.2
- new net: Q1.2 (B), R2.2
- new net VAC: K1.14, M?.1
- new net VCC: D1.1 (K), K1.2, U1.4
Changed lines of the file:
@@
 	5600 2950 5950 2950
 Wire Wire Line
-	5600 2850 5950 2850
-Wire Wire Line
 	5600 2650 5950 2650
 Wire Wire Line
@@
 	5600 2750 5700 2750
 Wire Wire Line
-	5700 2750 5700 4400
+	5700 2750 5700 3450
 Wire Wire Line
 	4700 3350 4700 3450
 Wire Wire Line
 	4700 3450 4700 4400
-Wire Notes Line
-	8500 500  8500 3450
-Wire Notes Line
-	8500 3450 11200 3450
 Wire Wire Line
 	4800 3050 4050 3050
 Text Notes 5100 2850 0    60   ~ 0
 1
+$Comp
+L Isolator:EL814 U1
+U 1 1 5EAAC487
+P 7700 2950
+F 0 "U1" H 7700 3275 50  0000 C CNN
+F 1 "EL814" H 7700 3184 50  0000 C CNN
+F 2 "" H 7500 2750 50  0001 L CIN
+F 3 "http://www.everlight.com/file/ProductFile/EL814.pdf" H 7725 2950 50  0001 L CNN
+	1    7700 2950
+	1    0    0    -1
+$EndComp
+$Comp
+L Device:R R1
+U 1 1 5EAAF00E
+P 6950 2850
+F 0 "R1" V 6743 2850 50  0000 C CNN
+F 1 "1000" V 6834 2850 50  0000 C CNN
+F 2 "" V 6880 2850 50  0001 C CNN
+F 3 "~" H 6950 2850 50  0001 C CNN
+	1    6950 2850
+	0    1    1    0
+$EndComp
+Wire Wire Line
+	7400 2850 7100 2850
+Wire Wire Line
+	5600 2850 6800 2850
+$Comp
+L Device:LED D?
+U 1 1 5EAB52F6
+P 7000 3450
+F 0 "D?" H 6993 3666 50  0000 C CNN
+F 1 "LED" H 6993 3575 50  0000 C CNN
+F 2 "" H 7000 3450 50  0001 C CNN
+F 3 "~" H 7000 3450 50  0001 C CNN
+	1    7000 3450
+	1    0    0    -1
+$EndComp
+Wire Wire Line
+	7400 3050 7200 3050
+Connection ~ 5700 3450
+Wire Wire Line
+	5700 3450 5700 4400
+Wire Wire Line
+	7200 3450 7150 3450
+Wire Wire Line
+	7200 3050 7200 3450
+Wire Wire Line
+	5700 3450 6850 3450
+$Comp
+L power:VCC #PWR0101
+U 1 1 5EABD3C3
+P 8150 2250
+F 0 "#PWR0101" H 8150 2100 50  0001 C CNN
+F 1 "VCC" H 8167 2423 50  0000 C CNN
+F 2 "" H 8150 2250 50  0001 C CNN
+F 3 "" H 8150 2250 50  0001 C CNN
+	1    8150 2250
+	1    0    0    -1
+$EndComp
+Wire Wire Line
+	8150 2250 8150 2850
+Wire Wire Line
+	8150 2850 8000 2850
+$Comp
+L Relay:DIPxx-1Cxx-51x K1
+U 1 1 5EAC1216
+P 9250 3050
+F 0 "K1" V 8683 3050 50  0000 C CNN
+F 1 "833H-1C-C 12V DC" V 8774 3050 50  0000 C CNN
+F 2 "Relay_THT:Relay_StandexMeder_DIP_LowProfile" H 9700 3000 50  0001 L CNN
+F 3 "https://www.mouser.cn/datasheet/2/378/20119191320287145-4912.pdf" H 9250 3050 50  0001 C CNN
+	1    9250 3050
+	0    1    1    0
+$EndComp
+Wire Wire Line
+	8950 2850 8550 2850
+Connection ~ 8150 2850
+$Comp
+L Diode:1N4007 D1
+U 1 1 5EAC7E2B
+P 8550 3100
+F 0 "D1" V 8504 3179 50  0000 L CNN
+F 1 "1N4007" V 8595 3179 50  0000 L CNN
+F 2 "Diode_THT:D_DO-41_SOD81_P10.16mm_Horizontal" H 8550 2925 50  0001 C CNN
+F 3 "http://www.vishay.com/docs/88503/1n4001.pdf" H 8550 3100 50  0001 C CNN
+	1    8550 3100
+	0    1    1    0
+$EndComp
+Wire Wire Line
+	8550 2950 8550 2850
+Connection ~ 8550 2850
+Wire Wire Line
+	8550 2850 8150 2850
+$Comp
+L Transistor_BJT:BC547 Q1
+U 1 1 5EACD121
+P 8550 4150
+F 0 "Q1" H 8741 4196 50  0000 L CNN
+F 1 "BC547" H 8741 4105 50  0000 L CNN
+F 2 "Package_TO_SOT_THT:TO-92_Inline" H 8750 4075 50  0001 L CIN
+F 3 "http://www.fairchildsemi.com/ds/BC/BC547.pdf" H 8550 4150 50  0001 L CNN
+	1    8550 4150
+	1    0    0    -1
+$EndComp
+$Comp
+L Device:R R2
+U 1 1 5EAD05F6
+P 8150 3600
+F 0 "R2" H 8220 3646 50  0000 L CNN
+F 1 "1000" H 8220 3555 50  0000 L CNN
+F 2 "" V 8080 3600 50  0001 C CNN
+F 3 "~" H 8150 3600 50  0001 C CNN
+	1    8150 3600
+	1    0    0    -1
+$EndComp
+Wire Wire Line
+	8350 4150 8150 4150
+Wire Wire Line
+	8150 4150 8150 3750
+Wire Wire Line
+	8150 3450 8150 3050
+Wire Wire Line
+	8150 3050 8000 3050
+$Comp
+L Motor:Motor_AC M?
+U 1 1 5EAD36B7
+P 10550 3100
+F 0 "M?" H 10708 3096 50  0000 L CNN
+F 1 "Motor_AC" H 10708 3005 50  0000 L CNN
+F 2 "" H 10550 3010 50  0001 C CNN
+F 3 "~" H 10550 3010 50  0001 C CNN
+	1    10550 3100
+	1    0    0    -1
+$EndComp
+$Comp
+L power:VAC #PWR0102
+U 1 1 5EAD5898
+P 10000 2200
+F 0 "#PWR0102" H 10000 2100 50  0001 C CNN
+F 1 "VAC" H 10000 2475 50  0000 C CNN
+F 2 "" H 10000 2200 50  0001 C CNN
+F 3 "" H 10000 2200 50  0001 C CNN
+	1    10000 2200
+	1    0    0    -1
+$EndComp
+$Comp
+L power:VAC #PWR0103
+U 1 1 5EAD6635
+P 10500 2200
+F 0 "#PWR0103" H 10500 2100 50  0001 C CNN
+F 1 "VAC" H 10500 2475 50  0000 C CNN
+F 2 "" H 10500 2200 50  0001 C CNN
+F 3 "" H 10500 2200 50  0001 C CNN
+	1    10500 2200
+	1    0    0    -1
+$EndComp
+Wire Wire Line
+	9550 2850 10000 2850
+Wire Wire Line
+	10000 2850 10000 3950
+Wire Wire Line
+	10000 3950 8650 3950
+Wire Wire Line
+	8650 3950 8550 3950
+Wire Wire Line
+	8550 3950 8550 3250
+Connection ~ 8650 3950
+Wire Wire Line
+	8950 3250 8950 3650
+Wire Wire Line
+	8950 3650 10550 3650
+Wire Wire Line
+	10550 3650 10550 3400
+Wire Wire Line
+	10550 2900 10550 2600
+Wire Wire Line
+	10550 2600 10500 2600
+Wire Wire Line
+	10500 2600 10500 2200
+Wire Wire Line
+	9550 3350 9800 3350
+Wire Wire Line
+	9800 3350 9800 2500
+Wire Wire Line
+	9800 2500 10000 2500
+Wire Wire Line
+	10000 2500 10000 2200
+Wire Wire Line
+	8650 4350 8650 4650
+Wire Wire Line
+	8650 4650 6750 4650
+Wire Wire Line
+	6750 4650 6750 4400
+Wire Wire Line
+	6750 4400 5700 4400
+Connection ~ 5700 4400
 $EndSCHEMATC

Commit message: Update Pressure-control.sch
Parts:
- removed K1: 833H-1C-C 12V DC, Relay_THT:Relay_StandexMeder_DIP_LowProfile, symbol Relay:DIPxx-1Cxx-51x
- added K?: 833H-1C-C-12VDC, 833H1CC12VDC, symbol SamacSys_Parts:833H-1C-C-12VDC
Connections:
- net VAC: now also K?.5 (COM)
- net VCC: now also K?.4 (COIL_2)
- net at D1.2 (A), Q1.1 (C): now also K?.1 (COIL_1)
- net at M?.2: now also K?.3 (NO)
Changed lines of the file:
@@
 Wire Wire Line
 	8150 2850 8000 2850
-$Comp
-L Relay:DIPxx-1Cxx-51x K1
-U 1 1 5EAC1216
-P 9250 3050
-F 0 "K1" V 8683 3050 50  0000 C CNN
-F 1 "833H-1C-C 12V DC" V 8774 3050 50  0000 C CNN
-F 2 "Relay_THT:Relay_StandexMeder_DIP_LowProfile" H 9700 3000 50  0001 L CNN
-F 3 "https://www.mouser.cn/datasheet/2/378/20119191320287145-4912.pdf" H 9250 3050 50  0001 C CNN
-	1    9250 3050
-	0    1    1    0
-$EndComp
-Wire Wire Line
-	8950 2850 8550 2850
 Connection ~ 8150 2850
 $Comp
@@
 $EndComp
 Wire Wire Line
-	9550 2850 10000 2850
-Wire Wire Line
-	10000 2850 10000 3950
-Wire Wire Line
-	10000 3950 8650 3950
-Wire Wire Line
 	8650 3950 8550 3950
 Wire Wire Line
 	8550 3950 8550 3250
-Connection ~ 8650 3950
-Wire Wire Line
-	8950 3250 8950 3650
-Wire Wire Line
-	8950 3650 10550 3650
-Wire Wire Line
-	10550 3650 10550 3400
-Wire Wire Line
-	10550 2900 10550 2600
-Wire Wire Line
-	10550 2600 10500 2600
-Wire Wire Line
-	10500 2600 10500 2200
-Wire Wire Line
-	9550 3350 9800 3350
-Wire Wire Line
-	9800 3350 9800 2500
-Wire Wire Line
-	9800 2500 10000 2500
 Wire Wire Line
 	10000 2500 10000 2200
@@
 	6750 4400 5700 4400
 Connection ~ 5700 4400
+$Comp
+L SamacSys_Parts:833H-1C-C-12VDC K?
+U 1 1 5EAB775F
+P 9400 4150
+F 0 "K?" V 10096 3822 50  0000 R CNN
+F 1 "833H-1C-C-12VDC" V 10005 3822 50  0000 R CNN
+F 2 "833H1CC12VDC" H 10550 4250 50  0001 L CNN
+F 3 "https://componentsearchengine.com/Datasheets/1/833H-1C-C-12VDC.pdf" H 10550 4150 50  0001 L CNN
+F 4 "General Purpose Relays 12Vdc 10A Sugar Cube" H 10550 4050 50  0001 L CNN "Description"
+F 5 "15" H 10550 3950 50  0001 L CNN "Height"
+F 6 "Song Chuan" H 10550 3850 50  0001 L CNN "Manufacturer_Name"
+F 7 "833H-1C-C-12VDC" H 10550 3750 50  0001 L CNN "Manufacturer_Part_Number"
+F 8 "893-833H-1C-C-12VDC" H 10550 3650 50  0001 L CNN "Mouser Part Number"
+F 9 "https://www.mouser.co.uk/ProductDetail/Song-Chuan/833H-1C-C-12VDC?qs=X4N6sOTYzkgmOWwYJwJPXg%3D%3D" H 10550 3550 50  0001 L CNN "Mouser Price/Stock"
+F 10 "" H 10550 3450 50  0001 L CNN "RS Part Number"
+F 11 "" H 10550 3350 50  0001 L CNN "RS Price/Stock"
+	1    9400 4150
+	0    -1   -1   0
+$EndComp
+Wire Wire Line
+	8550 2850 9400 2850
+Wire Wire Line
+	9400 4150 9050 4150
+Wire Wire Line
+	9050 4150 9050 3950
+Wire Wire Line
+	9050 3950 8650 3950
+Connection ~ 8650 3950
+Wire Wire Line
+	9500 2850 9500 2500
+Wire Wire Line
+	9500 2500 10000 2500
+Wire Wire Line
+	9600 4150 10550 4150
+Wire Wire Line
+	10550 3400 10550 4150
+Wire Wire Line
+	10550 2900 10500 2900
+Wire Wire Line
+	10500 2900 10500 2200
 $EndSCHEMATC

Commit message: Update Pressure-control.sch
Parts:
- removed K?: 833H-1C-C-12VDC, 833H1CC12VDC, symbol SamacSys_Parts:833H-1C-C-12VDC
- removed M?: Motor_AC, symbol Motor:Motor_AC
- added F1: 10A, symbol Device:Fuse
- added J1: DC_INPUT_12V, symbol Connector:Conn_01x02_Male
- added J2: DC_OUTPUT_12V, symbol Connector:Conn_01x02_Male
- added K1: SONGCHUAN-833H-1C-C-12VDC, 833H1CC12VDC, symbol Pressure-control-rescue:SONGCHUAN-833H-1C-C-12VDC
Connections:
- net GND: now also J1.2 (Pin_2), J2.2 (Pin_2)
- net at D1.2 (A), Q1.1 (C): now also F1.2, K1.2 (NC), K1.4
- net A0 renamed PRESSURE_SENSOR_OUTPUT
- net VCC: no longer names the net of D1.1 (K), U1.4
- net VCC: now also K1.1
- new net: J2.1 (Pin_1), K1.5 (COM), K1.6
- new net: F1.1, J1.1 (Pin_1)
Changed lines of the file:
@@
 Text Label 5950 2450 0    60   ~ 0
 A5(SCL)
-Text Notes 8550 750  0    60   ~ 0
+Text Notes 9250 800  0    60   ~ 0
 Shield for Arduino that uses\nthe same pin disposition\nlike "Uno" board Rev 3.
 $Comp
@@
 $EndComp
 Wire Notes Line
-	8525 825  9925 825
+	9225 875  10625 875
 Wire Notes Line
-	9925 825  9925 475
+	10625 875  10625 525
 Wire Wire Line
 	4750 2700 4750 2950
@@
 Wire Wire Line
 	4550 3150 4550 2700
-Wire Wire Line
-	4800 3750 4300 3750
 Wire Wire Line
 	4800 3850 4300 3850
@@
 	5700 3450 6850 3450
 $Comp
-L power:VCC #PWR0101
-U 1 1 5EABD3C3
-P 8150 2250
-F 0 "#PWR0101" H 8150 2100 50  0001 C CNN
-F 1 "VCC" H 8167 2423 50  0000 C CNN
-F 2 "" H 8150 2250 50  0001 C CNN
-F 3 "" H 8150 2250 50  0001 C CNN
-	1    8150 2250
-	1    0    0    -1
-$EndComp
-Wire Wire Line
-	8150 2250 8150 2850
-Wire Wire Line
-	8150 2850 8000 2850
-Connection ~ 8150 2850
-$Comp
 L Diode:1N4007 D1
 U 1 1 5EAC7E2B
@@
 Wire Wire Line
 	8550 2950 8550 2850
-Connection ~ 8550 2850
-Wire Wire Line
-	8550 2850 8150 2850
 $Comp
 L Transistor_BJT:BC547 Q1
@@
 Wire Wire Line
 	8150 3050 8000 3050
-$Comp
-L Motor:Motor_AC M?
-U 1 1 5EAD36B7
-P 10550 3100
-F 0 "M?" H 10708 3096 50  0000 L CNN
-F 1 "Motor_AC" H 10708 3005 50  0000 L CNN
-F 2 "" H 10550 3010 50  0001 C CNN
-F 3 "~" H 10550 3010 50  0001 C CNN
-	1    10550 3100
-	1    0    0    -1
-$EndComp
-$Comp
-L power:VAC #PWR0102
-U 1 1 5EAD5898
-P 10000 2200
-F 0 "#PWR0102" H 10000 2100 50  0001 C CNN
-F 1 "VAC" H 10000 2475 50  0000 C CNN
-F 2 "" H 10000 2200 50  0001 C CNN
-F 3 "" H 10000 2200 50  0001 C CNN
-	1    10000 2200
-	1    0    0    -1
-$EndComp
-$Comp
-L power:VAC #PWR0103
-U 1 1 5EAD6635
-P 10500 2200
-F 0 "#PWR0103" H 10500 2100 50  0001 C CNN
-F 1 "VAC" H 10500 2475 50  0000 C CNN
-F 2 "" H 10500 2200 50  0001 C CNN
-F 3 "" H 10500 2200 50  0001 C CNN
-	1    10500 2200
-	1    0    0    -1
-$EndComp
-Wire Wire Line
-	8650 3950 8550 3950
-Wire Wire Line
-	8550 3950 8550 3250
-Wire Wire Line
-	10000 2500 10000 2200
-Wire Wire Line
-	8650 4350 8650 4650
-Wire Wire Line
-	8650 4650 6750 4650
-Wire Wire Line
-	6750 4650 6750 4400
-Wire Wire Line
-	6750 4400 5700 4400
 Connection ~ 5700 4400
 $Comp
-L SamacSys_Parts:833H-1C-C-12VDC K?
-U 1 1 5EAB775F
-P 9400 4150
-F 0 "K?" V 10096 3822 50  0000 R CNN
-F 1 "833H-1C-C-12VDC" V 10005 3822 50  0000 R CNN
-F 2 "833H1CC12VDC" H 10550 4250 50  0001 L CNN
-F 3 "https://componentsearchengine.com/Datasheets/1/833H-1C-C-12VDC.pdf" H 10550 4150 50  0001 L CNN
-F 4 "General Purpose Relays 12Vdc 10A Sugar Cube" H 10550 4050 50  0001 L CNN "Description"
-F 5 "15" H 10550 3950 50  0001 L CNN "Height"
-F 6 "Song Chuan" H 10550 3850 50  0001 L CNN "Manufacturer_Name"
-F 7 "833H-1C-C-12VDC" H 10550 3750 50  0001 L CNN "Manufacturer_Part_Number"
-F 8 "893-833H-1C-C-12VDC" H 10550 3650 50  0001 L CNN "Mouser Part Number"
-F 9 "https://www.mouser.co.uk/ProductDetail/Song-Chuan/833H-1C-C-12VDC?qs=X4N6sOTYzkgmOWwYJwJPXg%3D%3D" H 10550 3550 50  0001 L CNN "Mouser Price/Stock"
-F 10 "" H 10550 3450 50  0001 L CNN "RS Part Number"
-F 11 "" H 10550 3350 50  0001 L CNN "RS Price/Stock"
-	1    9400 4150
-	0    -1   -1   0
-$EndComp
-Wire Wire Line
-	8550 2850 9400 2850
-Wire Wire Line
-	9400 4150 9050 4150
-Wire Wire Line
-	9050 4150 9050 3950
-Wire Wire Line
-	9050 3950 8650 3950
-Connection ~ 8650 3950
-Wire Wire Line
-	9500 2850 9500 2500
-Wire Wire Line
-	9500 2500 10000 2500
-Wire Wire Line
-	9600 4150 10550 4150
-Wire Wire Line
-	10550 3400 10550 4150
-Wire Wire Line
-	10550 2900 10500 2900
-Wire Wire Line
-	10500 2900 10500 2200
+L Pressure-control-rescue:SONGCHUAN-833H-1C-C-12VDC K1
+U 1 1 5EAD35C2
+P 9450 2900
+F 0 "K1" V 9033 2900 50  0000 C CNN
+F 1 "SONGCHUAN-833H-1C-C-12VDC" V 9124 2900 50  0000 C CNN
+F 2 "833H1CC12VDC" H 10250 3150 50  0001 L CNN
+F 3 "https://componentsearchengine.com/Datasheets/1/833H-1C-C-12VDC.pdf" H 10250 3050 50  0001 L CNN
+F 4 "General Purpose Relays 12Vdc 10A Sugar Cube" H 10250 2950 50  0001 L CNN "Description"
+F 5 "15" H 10250 2850 50  0001 L CNN "Height"
+F 6 "Song Chuan" H 10250 2750 50  0001 L CNN "Manufacturer_Name"
+F 7 "833H-1C-C-12VDC" H 10250 2650 50  0001 L CNN "Manufacturer_Part_Number"
+F 8 "893-833H-1C-C-12VDC" H 10250 2550 50  0001 L CNN "Mouser Part Number"
+F 9 "https://www.mouser.co.uk/ProductDetail/Song-Chuan/833H-1C-C-12VDC?qs=X4N6sOTYzkgmOWwYJwJPXg%3D%3D" H 10250 2450 50  0001 L CNN "Mouser Price/Stock"
+	1    9450 2900
+	0    1    1    0
+$EndComp
+Wire Wire Line
+	9150 2850 8550 2850
+Connection ~ 8550 2850
+Wire Wire Line
+	8650 3950 8650 3600
+Wire Wire Line
+	8650 3600 9000 3600
+Wire Wire Line
+	9000 3600 9000 2250
+Wire Wire Line
+	9000 2250 10250 2250
+Wire Wire Line
+	10250 2250 10250 2850
+Wire Wire Line
+	10250 2850 9750 2850
+Wire Wire Line
+	8650 3600 8550 3600
+Wire Wire Line
+	8550 3600 8550 3250
+Connection ~ 8650 3600
+$Comp
+L Connector:Conn_01x02_Male J1
+U 1 1 5EAE9078
+P 10800 3150
+F 0 "J1" H 10908 3331 50  0000 C CNN
+F 1 "DC_INPUT_12V" H 10908 3240 50  0000 C CNN
+F 2 "" H 10800 3150 50  0001 C CNN
+F 3 "~" H 10800 3150 50  0001 C CNN
+	1    10800 3150
+	-1   0    0    -1
+$EndComp
+$Comp
+L Connector:Conn_01x02_Male J2
+U 1 1 5EAF2928
+P 10800 4000
+F 0 "J2" H 10908 4181 50  0000 C CNN
+F 1 "DC_OUTPUT_12V" H 10908 4090 50  0000 C CNN
+F 2 "" H 10800 4000 50  0001 C CNN
+F 3 "~" H 10800 4000 50  0001 C CNN
+	1    10800 4000
+	-1   0    0    -1
+$EndComp
+Wire Wire Line
+	10600 4000 9150 4000
+Wire Wire Line
+	9150 4000 9150 3250
+Wire Wire Line
+	10600 3250 10250 3250
+Wire Wire Line
+	10250 3250 10250 4100
+Wire Wire Line
+	10250 4100 10600 4100
+Wire Wire Line
+	10250 4100 10250 4600
+Connection ~ 10250 4100
+$Comp
+L power:GND #PWR?
+U 1 1 5EAFB94C
+P 10250 4600
+F 0 "#PWR?" H 10250 4350 50  0001 C CNN
+F 1 "GND" H 10255 4427 50  0000 C CNN
+F 2 "" H 10250 4600 50  0001 C CNN
+F 3 "" H 10250 4600 50  0001 C CNN
+	1    10250 4600
+	1    0    0    -1
+$EndComp
+Wire Wire Line
+	10250 2850 10250 3150
+Wire Wire Line
+	9750 3150 10250 3150
+Connection ~ 10250 2850
+Wire Wire Line
+	8000 2850 8550 2850
+$Comp
+L Device:Fuse F1
+U 1 1 5EAFE39A
+P 10400 3150
+F 0 "F1" V 10203 3150 50  0000 C CNN
+F 1 "10A" V 10294 3150 50  0000 C CNN
+F 2 "" V 10330 3150 50  0001 C CNN
+F 3 "~" H 10400 3150 50  0001 C CNN
+	1    10400 3150
+	0    1    1    0
+$EndComp
+Connection ~ 10250 3150
+Wire Wire Line
+	10600 3150 10550 3150
+Wire Wire Line
+	3050 3750 4800 3750
+Text GLabel 3050 3750 0    50   Input ~ 0
+PRESSURE_SENSOR_OUTPUT
+Wire Wire Line
+	8650 4400 8650 4350
+Wire Wire Line
+	5700 4400 8650 4400
 $EndSCHEMATC
